Commit message: moveit integration

File: robotic_arm/urdf/Robot_Arm.xacro (robot description, xacro)
@@ -84,4 +84,5 @@
     name="base_waist_joint"
     type="revolute">
+    <dynamics damping="1.0" friction="1.0"/>
     <origin
       xyz="0 0 0.0575"
@@ -142,4 +143,5 @@
     name="waist_arm_joint"
     type="revolute">
+    <dynamics damping="1.0" friction="1.0"/>
     <origin
       xyz="0 0.04028 -0.01391"
@@ -200,4 +202,5 @@
     name="arm_end_joint"
     type="revolute">
+    <dynamics damping="1.0" friction="1.0"/>
     <origin
       xyz="0 0.12 0"
@@ -258,4 +261,5 @@
     name="end_support_joint"
     type="fixed">
+    <dynamics damping="1.0" friction="1.0"/>
     <origin
       xyz="0.065057 -0.0082418 -0.011"
@@ -268,3 +272,123 @@
       xyz="0 0 0" />
   </joint>
+  <link
+    name="cam_Link">
+    <inertial>
+      <origin
+        xyz="0.0215 0.0215 0.0215"
+        rpy="0 0 0" />
+      <mass
+        value="0.079507" />
+      <inertia
+        ixx="2.4501E-05"
+        ixy="-1.8211E-21"
+        ixz="-5.7909E-22"
+        iyy="2.4501E-05"
+        iyz="-2.7946E-23"
+        izz="2.4501E-05" />
+    </inertial>
+    <visual>
+      <origin
+        xyz="0 0 0"
+        rpy="0 0 0" />
+      <geometry>
+        <mesh
+          filename="file:///home/khaled/ros2_ws/src/robotic_arm/meshes/cam_Link.STL" />
+      </geometry>
+      <material
+        name="">
+        <color
+          rgba="0.79216 0.81961 0.93333 1" />
+      </material>
+    </visual>
+    <collision>
+      <origin
+        xyz="0 0 0"
+        rpy="0 0 0" />
+      <geometry>
+        <mesh
+          filename="file:///home/khaled/ros2_ws/src/robotic_arm/meshes/cam_Link.STL" />
+      </geometry>
+    </collision>
+  </link>
+  <joint
+    name="support_cam_joint"
+    type="fixed">
+    <dynamics damping="1.0" friction="1.0"/>
+    <origin
+      xyz="-0.0028878 0.074628 0.023"
+      rpy="-1.5708 0 -1.5708" />
+    <parent
+      link="support_Link" />
+    <child
+      link="cam_Link" />
+    <axis
+      xyz="0 0 0" />
+  </joint>
+  <!-- Robot Tip -->
+  <link name="tip_link"/>
+  <joint name="support_tip_joint" type="fixed">
+    <parent link="support_Link"/>
+    <child link="tip_link"/>
+    <origin xyz="0.025 0.004 0.001" rpy="0 0 0"/>
+  </joint>
+  <xacro:macro name="control" params="joint">
+    <transmission name="${joint}_transmission">
+      <type>transmission_interface/SimpleTransmission</type>
+      <joint name="${joint}">
+        <hardwareInterface>position</hardwareInterface>
+      </joint>
+      <actuator name="${joint}_motor">
+        <hardwareInterface>position</hardwareInterface>
+        <mechanicalReduction>1</mechanicalReduction>
+      </actuator>
+    </transmission>
+  </xacro:macro>
+<!-- Usage -->
+  <xacro:control joint="base_waist_joint"/>
+  <xacro:control joint="waist_arm_joint"/>
+  <xacro:control joint="arm_end_joint"/>
+  <xacro:control joint="end_support_joint"/>
+  <xacro:control joint="support_cam_joint"/>
+  <gazebo>
+    <plugin name="gazebo_ros2_control" filename="libgazebo_ros2_control.so">
+      <robotNamespace>/robotic_arm</robotNamespace>
+      <parameters>$(find moveit_robotic_arm)/config/ros2_controllers.yaml</parameters>
+    </plugin>
+  </gazebo>
+  <ros2_control name="controller_manager" type="system">
+    <hardware>
+      <plugin>gazebo_ros2_control/GazeboSystem</plugin>
+    </hardware>
+    <joint>
+      <name>base_waist_joint</name>
+      <command_interface>position</command_interface>
+      <state_interface>position</state_interface>
+      <state_interface>velocity</state_interface>
+    </joint>
+    <joint>
+      <name>waist_arm_joint</name>
+      <command_interface>position</command_interface>
+      <state_interface>position</state_interface>
+      <state_interface>velocity</state_interface>
+    </joint>
+    <joint>
+      <name>arm_end_joint</name>
+      <command_interface>position</command_interface>
+      <state_interface>position</state_interface>
+      <state_interface>velocity</state_interface>
+    </joint>
+    <joint>
+      <name>end_support_joint</name>
+      <command_interface>position</command_interface>
+      <state_interface>position</state_interface>
+      <state_interface>velocity</state_interface>
+    </joint>
+    <joint>
+      <name>support_cam_joint</name>
+      <command_interface>position</command_interface>
+      <state_interface>position</state_interface>
+      <state_interface>velocity</state_interface>
+    </joint>
+  </ros2_control>
 </robot>

Commit message: fix

File: robotic_arm/urdf/Robot_Arm.xacro (robot description, xacro)
@@ -84,5 +84,4 @@
     name="base_waist_joint"
     type="revolute">
-    <dynamics damping="1.0" friction="1.0"/>
     <origin
       xyz="0 0 0.0575"
@@ -143,5 +142,4 @@
     name="waist_arm_joint"
     type="revolute">
-    <dynamics damping="1.0" friction="1.0"/>
     <origin
       xyz="0 0.04028 -0.01391"
@@ -202,5 +200,4 @@
     name="arm_end_joint"
     type="revolute">
-    <dynamics damping="1.0" friction="1.0"/>
     <origin
       xyz="0 0.12 0"
@@ -261,5 +258,4 @@
     name="end_support_joint"
     type="fixed">
-    <dynamics damping="1.0" friction="1.0"/>
     <origin
       xyz="0.065057 -0.0082418 -0.011"
@@ -272,123 +268,3 @@
       xyz="0 0 0" />
   </joint>
-  <link
-    name="cam_Link">
-    <inertial>
-      <origin
-        xyz="0.0215 0.0215 0.0215"
-        rpy="0 0 0" />
-      <mass
-        value="0.079507" />
-      <inertia
-        ixx="2.4501E-05"
-        ixy="-1.8211E-21"
-        ixz="-5.7909E-22"
-        iyy="2.4501E-05"
-        iyz="-2.7946E-23"
-        izz="2.4501E-05" />
-    </inertial>
-    <visual>
-      <origin
-        xyz="0 0 0"
-        rpy="0 0 0" />
-      <geometry>
-        <mesh
-          filename="file:///home/khaled/ros2_ws/src/robotic_arm/meshes/cam_Link.STL" />
-      </geometry>
-      <material
-        name="">
-        <color
-          rgba="0.79216 0.81961 0.93333 1" />
-      </material>
-    </visual>
-    <collision>
-      <origin
-        xyz="0 0 0"
-        rpy="0 0 0" />
-      <geometry>
-        <mesh
-          filename="file:///home/khaled/ros2_ws/src/robotic_arm/meshes/cam_Link.STL" />
-      </geometry>
-    </collision>
-  </link>
-  <joint
-    name="support_cam_joint"
-    type="fixed">
-    <dynamics damping="1.0" friction="1.0"/>
-    <origin
-      xyz="-0.0028878 0.074628 0.023"
-      rpy="-1.5708 0 -1.5708" />
-    <parent
-      link="support_Link" />
-    <child
-      link="cam_Link" />
-    <axis
-      xyz="0 0 0" />
-  </joint>
-  <!-- Robot Tip -->
-  <link name="tip_link"/>
-  <joint name="support_tip_joint" type="fixed">
-    <parent link="support_Link"/>
-    <child link="tip_link"/>
-    <origin xyz="0.025 0.004 0.001" rpy="0 0 0"/>
-  </joint>
-  <xacro:macro name="control" params="joint">
-    <transmission name="${joint}_transmission">
-      <type>transmission_interface/SimpleTransmission</type>
-      <joint name="${joint}">
-        <hardwareInterface>position</hardwareInterface>
-      </joint>
-      <actuator name="${joint}_motor">
-        <hardwareInterface>position</hardwareInterface>
-        <mechanicalReduction>1</mechanicalReduction>
-      </actuator>
-    </transmission>
-  </xacro:macro>
-<!-- Usage -->
-  <xacro:control joint="base_waist_joint"/>
-  <xacro:control joint="waist_arm_joint"/>
-  <xacro:control joint="arm_end_joint"/>
-  <xacro:control joint="end_support_joint"/>
-  <xacro:control joint="support_cam_joint"/>
-  <gazebo>
-    <plugin name="gazebo_ros2_control" filename="libgazebo_ros2_control.so">
-      <robotNamespace>/robotic_arm</robotNamespace>
-      <parameters>$(find moveit_robotic_arm)/config/ros2_controllers.yaml</parameters>
-    </plugin>
-  </gazebo>
-  <ros2_control name="controller_manager" type="system">
-    <hardware>
-      <plugin>gazebo_ros2_control/GazeboSystem</plugin>
-    </hardware>
-    <joint>
-      <name>base_waist_joint</name>
-      <command_interface>position</command_interface>
-      <state_interface>position</state_interface>
-      <state_interface>velocity</state_interface>
-    </joint>
-    <joint>
-      <name>waist_arm_joint</name>
-      <command_interface>position</command_interface>
-      <state_interface>position</state_interface>
-      <state_interface>velocity</state_interface>
-    </joint>
-    <joint>
-      <name>arm_end_joint</name>
-      <command_interface>position</command_interface>
-      <state_interface>position</state_interface>
-      <state_interface>velocity</state_interface>
-    </joint>
-    <joint>
-      <name>end_support_joint</name>
-      <command_interface>position</command_interface>
-      <state_interface>position</state_interface>
-      <state_interface>velocity</state_interface>
-    </joint>
-    <joint>
-      <name>support_cam_joint</name>
-      <command_interface>position</command_interface>
-      <state_interface>position</state_interface>
-      <state_interface>velocity</state_interface>
-    </joint>
-  </ros2_control>
 </robot>

Commit message: fix

File: robotic_arm/urdf/Robot_Arm.xacro (robot description, xacro)
@@ -1,4 +1,6 @@
 <?xml version="1.0" encoding="utf-8"?>
 <robot name="robotic_arm" xmlns:xacro="http:///www.ros.org/wiki/xacro">
+  <xacro:include filename="$(find robotic_arm)/urdf/Robot_Arm_control.xacro" />
+  <xacro:include filename="$(find robotic_arm)/urdf/Robot_Arm_gazebo.xacro" />
   <link
     name="base_link">
@@ -23,5 +25,5 @@
       <geometry>
         <mesh
-          filename="file:///home/khaled/ros2_ws/src/robotic_arm/meshes/base_link.STL" />
+          filename="package://robotic_arm/meshes/base_link.STL" />
       </geometry>
       <material
@@ -37,5 +39,5 @@
       <geometry>
         <mesh
-          filename="file:///home/khaled/ros2_ws/src/robotic_arm/meshes/base_link.STL" />
+          filename="package://robotic_arm/meshes/base_link.STL" />
       </geometry>
     </collision>
@@ -63,5 +65,5 @@
       <geometry>
         <mesh
-          filename="file:///home/khaled/ros2_ws/src/robotic_arm/meshes/waist_Link.STL" />
+          filename="package://robotic_arm/meshes/waist_Link.STL" />
       </geometry>
       <material
@@ -77,5 +79,5 @@
       <geometry>
         <mesh
-          filename="file:///home/khaled/ros2_ws/src/robotic_arm/meshes/waist_Link.STL" />
+          filename="package://robotic_arm/meshes/waist_Link.STL" />
       </geometry>
     </collision>
@@ -121,5 +123,5 @@
       <geometry>
         <mesh
-          filename="file:///home/khaled/ros2_ws/src/robotic_arm/meshes/arm_Link.STL" />
+          filename="package://robotic_arm/meshes/arm_Link.STL" />
       </geometry>
       <material
@@ -135,5 +137,5 @@
       <geometry>
         <mesh
-          filename="file:///home/khaled/ros2_ws/src/robotic_arm/meshes/arm_Link.STL" />
+          filename="package://robotic_arm/meshes/arm_Link.STL" />
       </geometry>
     </collision>
@@ -179,5 +181,5 @@
       <geometry>
         <mesh
-          filename="file:///home/khaled/ros2_ws/src/robotic_arm/meshes/end_Link.STL" />
+          filename="package://robotic_arm/meshes/end_Link.STL" />
       </geometry>
       <material
@@ -193,5 +195,5 @@
       <geometry>
         <mesh
-          filename="file:///home/khaled/ros2_ws/src/robotic_arm/meshes/end_Link.STL" />
+          filename="package://robotic_arm/meshes/end_Link.STL" />
       </geometry>
     </collision>
@@ -237,5 +239,5 @@
       <geometry>
         <mesh
-          filename="file:///home/khaled/ros2_ws/src/robotic_arm/meshes/support_Link.STL" />
+          filename="package://robotic_arm/meshes/support_Link.STL" />
       </geometry>
       <material
@@ -251,5 +253,5 @@
       <geometry>
         <mesh
-          filename="file:///home/khaled/ros2_ws/src/robotic_arm/meshes/support_Link.STL" />
+          filename="package://robotic_arm/meshes/support_Link.STL" />
       </geometry>
     </collision>
@@ -268,3 +270,82 @@
       xyz="0 0 0" />
   </joint>
+  <link
+    name="cam_Link">
+    <inertial>
+      <origin
+        xyz="0.0215 0.0215 0.0215"
+        rpy="0 0 0" />
+      <mass
+        value="0.079507" />
+      <inertia
+        ixx="2.4501E-05"
+        ixy="-1.8211E-21"
+        ixz="-5.7909E-22"
+        iyy="2.4501E-05"
+        iyz="-2.7946E-23"
+        izz="2.4501E-05" />
+    </inertial>
+    <visual>
+      <origin
+        xyz="0 0 0"
+        rpy="0 0 0" />
+      <geometry>
+        <mesh
+          filename="package://robotic_arm/meshes/cam_Link.STL" />
+      </geometry>
+      <material
+        name="">
+        <color
+          rgba="0.79216 0.81961 0.93333 1" />
+      </material>
+    </visual>
+    <collision>
+      <origin
+        xyz="0 0 0"
+        rpy="0 0 0" />
+      <geometry>
+        <mesh
+          filename="package://robotic_arm/meshes/cam_Link.STL" />
+      </geometry>
+    </collision>
+  </link>
+  <joint
+    name="support_cam_joint"
+    type="fixed">
+    <origin
+      xyz="-0.0028878 0.074628 0.023"
+      rpy="-1.5708 0 -1.5708" />
+    <parent
+      link="support_Link" />
+    <child
+      link="cam_Link" />
+    <axis
+      xyz="0 0 0" />
+  </joint>
+  <!-- Robot Tip -->
+  <link name="tip_link"/>
+  <joint name="support_tip_joint" type="fixed">
+    <parent link="support_Link"/>
+    <child link="tip_link"/>
+    <origin xyz="0.025 0.004 0.001" rpy="0 0 0"/>
+  </joint>
+  <xacro:macro name="control" params="joint">
+    <transmission name="${joint}_transmission">
+      <plugin>transmission_interface/SimpleTransmission</plugin >
+      <joint name="${joint}_joint">
+        <hardwareInterface>position</hardwareInterface>
+        <mechanicalReduction>1.0</mechanicalReduction>
+      </joint>
+      <actuator name="${joint}_motor">
+        <hardwareInterface>position</hardwareInterface>
+        <mechanicalReduction>1.0</mechanicalReduction>
+      </actuator>
+    </transmission>
+  </xacro:macro>
+<!-- Usage -->
+  <xacro:control joint="base_waist"/>
+  <xacro:control joint="waist_arm"/>
+  <xacro:control joint="arm_end"/>
+  <xacro:control joint="end_support"/>
+  <xacro:control joint="support_cam"/>
 </robot>

Commit message: moveit bug fix & cam addition

File: robotic_arm/urdf/Robot_Arm.xacro (robot description, xacro)
@@ -274,5 +274,5 @@
     <inertial>
       <origin
-        xyz="0.0215 0.0215 0.0215"
+        xyz="-0.04 -0.022 -0.021"
         rpy="0 0 0" />
       <mass
@@ -288,5 +288,5 @@
     <visual>
       <origin
-        xyz="0 0 0"
+        xyz="-0.04 -0.022 -0.021"
         rpy="0 0 0" />
       <geometry>
@@ -314,6 +314,6 @@
     type="fixed">
     <origin
-      xyz="-0.0028878 0.074628 0.023"
-      rpy="-1.5708 0 -1.5708" />
+      xyz="0.04 0.0525 0.0005"
+      rpy="-1.570 0 0" />
     <parent
       link="support_Link" />
@@ -347,5 +347,24 @@
   <xacro:control joint="waist_arm"/>
   <xacro:control joint="arm_end"/>
-  <xacro:control joint="end_support"/>
-  <xacro:control joint="support_cam"/>
+  <link name="cam_Link_optical">
+    </link>
+    <joint name="cam_Link_joint" type="fixed">
+        <!-- these values have to be these values otherwise the gazebo camera
+            image won't be aligned properly with the frame it is supposedly
+            originating from -->
+        <origin xyz="0 0 0" rpy="${-pi/2} 0 ${-pi/2}"/>
+        <parent link="cam_Link"/>
+        <child link="cam_Link_optical"/>
+    </joint>
+    <gazebo reference="cam_Link">
+        <material>Gazebo/Red</material>
+        <sensor name="camera_sensor" type="camera">
+            <pose>0 0 0 0 0 0</pose>
+            <visualize>true</visualize>
+            <update_rate>10.0</update_rate>
+            <plugin name="camera_controller" filename="libgazebo_ros_camera.so">
+                <frame_name>cam_link_optical</frame_name>
+            </plugin>
+        </sensor>
+    </gazebo>
 </robot>

File: robotic_arm/urdf/Robot_Arm_control.xacro (robot description, xacro)
@@ -27,14 +27,4 @@
             <state_interface name="position"/>
         </joint>
-        <joint name="end_support_joint">
-            <command_interface name="position">
-            </command_interface>
-            <state_interface name="position"/>
-        </joint>
-        <joint name="support_cam_joint">
-            <command_interface name="position">
-            </command_interface>
-            <state_interface name="position"/>
-        </joint>
     </ros2_control>
 </robot>

Commit message: xyz coordinates

File: robotic_arm/urdf/Robot_Arm.xacro (robot description, xacro)
@@ -10,5 +10,5 @@
         rpy="0 0 0" />
       <mass
-        value="0.10728" />
+        value="0.83" />
       <inertia
         ixx="0.00014427"
@@ -368,3 +368,6 @@
         </sensor>
     </gazebo>
+    <gazebo reference="base_Link">
+        <material>Gazebo/Red</material>
+    </gazebo>
 </robot>

Commit message: fix base

File: robotic_arm/urdf/Robot_Arm.xacro (robot description, xacro)
@@ -329,4 +329,11 @@
     <child link="tip_link"/>
     <origin xyz="0.025 0.004 0.001" rpy="0 0 0"/>
+  </joint>
+  <!-- fix the robot to the world -->
+  <link name="world"/>
+  <joint name="world_fixed_joint" type="fixed">
+    <parent link="world"/>
+    <child link="base_link"/>
+    <origin xyz="0 0 0" rpy="0 0 0"/>
   </joint>
   <xacro:macro name="control" params="joint">
@@ -343,5 +350,4 @@
     </transmission>
   </xacro:macro>
-<!-- Usage -->
   <xacro:control joint="base_waist"/>
   <xacro:control joint="waist_arm"/>
@@ -350,7 +356,4 @@
     </link>
     <joint name="cam_Link_joint" type="fixed">
-        <!-- these values have to be these values otherwise the gazebo camera
-            image won't be aligned properly with the frame it is supposedly
-            originating from -->
         <origin xyz="0 0 0" rpy="${-pi/2} 0 ${-pi/2}"/>
         <parent link="cam_Link"/>
@@ -368,6 +371,3 @@
         </sensor>
     </gazebo>
-    <gazebo reference="base_Link">
-        <material>Gazebo/Red</material>
-    </gazebo>
 </robot>

Commit message: convertion to velocity

File: robotic_arm/urdf/Robot_Arm.xacro (robot description, xacro)
@@ -1,4 +1,6 @@
 <?xml version="1.0" encoding="utf-8"?>
 <robot name="robotic_arm" xmlns:xacro="http:///www.ros.org/wiki/xacro">
+  <xacro:include filename="$(find robotic_arm)/urdf/Robot_Arm_control.xacro" />
+  <xacro:include filename="$(find robotic_arm)/urdf/Robot_Arm_gazebo.xacro" />
   <link
     name="base_link">
@@ -8,5 +10,5 @@
         rpy="0 0 0" />
       <mass
-        value="0.10728" />
+        value="0.83" />
       <inertia
         ixx="0.00014427"
@@ -268,3 +270,109 @@
       xyz="0 0 0" />
   </joint>
+  <link
+    name="cam_Link">
+    <inertial>
+      <origin
+        xyz="-0.04 -0.022 -0.021"
+        rpy="0 0 0" />
+      <mass
+        value="0.079507" />
+      <inertia
+        ixx="2.4501E-05"
+        ixy="-1.8211E-21"
+        ixz="-5.7909E-22"
+        iyy="2.4501E-05"
+        iyz="-2.7946E-23"
+        izz="2.4501E-05" />
+    </inertial>
+    <visual>
+      <origin
+        xyz="-0.04 -0.022 -0.021"
+        rpy="0 0 0" />
+      <geometry>
+        <mesh
+          filename="file:///home/khaled/ros2_ws/src/robotic_arm/meshes/cam_Link.STL" />
+      </geometry>
+      <material
+        name="">
+        <color
+          rgba="0.79216 0.81961 0.93333 1" />
+      </material>
+    </visual>
+    <collision>
+      <origin
+        xyz="0 0 0"
+        rpy="0 0 0" />
+      <geometry>
+        <mesh
+          filename="file:///home/khaled/ros2_ws/src/robotic_arm/meshes/cam_Link.STL" />
+      </geometry>
+    </collision>
+  </link>
+  <joint
+    name="support_cam_joint"
+    type="fixed">
+    <origin
+      xyz="0.04 0.0525 0.0005"
+      rpy="-1.570 0 0" />
+    <parent
+      link="support_Link" />
+    <child
+      link="cam_Link" />
+    <axis
+      xyz="0 0 0" />
+  </joint>
+  <!-- Robot Tip -->
+  <link name="tip_link"/>
+  <joint name="support_tip_joint" type="fixed">
+    <parent link="support_Link"/>
+    <child link="tip_link"/>
+    <origin xyz="0.025 0.004 0.001" rpy="0 0 0"/>
+  </joint>
+  <!-- fix the robot to the world -->
+  <xacro:macro name="control" params="joint">
+    <transmission name="${joint}_transmission">
+      <plugin>transmission_interface/SimpleTransmission</plugin>
+      <joint name="${joint}_joint">
+        <hardwareInterface>hardware_interface/VelocityJointInterface</hardwareInterface>
+        <mechanicalReduction>1.0</mechanicalReduction>
+      </joint>
+      <actuator name="${joint}_motor">
+        <hardwareInterface>hardware_interface/VelocityJointInterface</hardwareInterface>
+        <mechanicalReduction>1.0</mechanicalReduction>
+      </actuator>
+    </transmission>
+  </xacro:macro>
+  <xacro:control joint="base_waist"/>
+  <xacro:control joint="waist_arm"/>
+  <xacro:control joint="arm_end"/>
+  <link name="cam_Link_optical">
+    </link>
+    <joint name="cam_Link_joint" type="fixed">
+        <origin xyz="0 0 0" rpy="${-pi/2} 0 ${-pi/2}"/>
+        <parent link="cam_Link"/>
+        <child link="cam_Link_optical"/>
+    </joint>
+    <gazebo reference="cam_Link">
+        <material>Gazebo/Red</material>
+        <sensor name="camera_sensor" type="camera">
+            <pose>0 0 0 0 0 0</pose>
+            <visualize>true</visualize>
+            <update_rate>10.0</update_rate>
+            <camera name="cam">
+              <horizontal_fov>1.3962634</horizontal_fov>
+              <image>
+                <width>1280</width>
+                <height>1280</height>
+                <format>R8G8B8</format>
+              </image>
+            </camera>
+            <plugin name="camera_controller" filename="libgazebo_ros_camera.so">
+                <frame_name>cam_link_optical</frame_name>
+                <image_width>1280</image_width>
+                <image_height>1280</image_height>
+                <update_rate>10.0</update_rate>
+            </plugin>
+        </sensor>
+    </gazebo>
 </robot>
