Commit message: ignition/velocity

File: robotic_arm/urdf/Robot_Arm.xacro (robot description, xacro)
@@ -1,6 +1,13 @@
 <?xml version="1.0" encoding="utf-8"?>
 <robot name="robotic_arm" xmlns:xacro="http:///www.ros.org/wiki/xacro">
-  <xacro:include filename="$(find robotic_arm)/urdf/Robot_Arm_control.xacro" />
-  <xacro:include filename="$(find robotic_arm)/urdf/Robot_Arm_gazebo.xacro" />
+  <xacro:property name="use_ignition" default="false"/>
+  <xacro:include filename="$(find robotic_arm)/urdf/Robot_Arm_control.xacro"/>
+  <xacro:include filename="$(find robotic_arm)/urdf/Robot_Arm_gazebo.xacro"/>
+  <xacro:if value="${use_ignition}">
+    <xacro:property name="mesh_dir" value="/home/khaled/ros2_ws/src/robotic_arm/meshes"/>
+  </xacro:if>
+  <xacro:unless value="${use_ignition}">
+    <xacro:property name="mesh_dir" value="package://robotic_arm/meshes"/>
+  </xacro:unless>
   <link
     name="base_link">
@@ -25,5 +32,5 @@
       <geometry>
         <mesh
-          filename="package://robotic_arm/meshes/base_link.STL" />
+          filename="${mesh_dir}/base_link.STL" />
       </geometry>
       <material
@@ -39,5 +46,5 @@
       <geometry>
         <mesh
-          filename="package://robotic_arm/meshes/base_link.STL" />
+          filename="${mesh_dir}/base_link.STL" />
       </geometry>
     </collision>
@@ -65,5 +72,5 @@
       <geometry>
         <mesh
-          filename="package://robotic_arm/meshes/waist_Link.STL" />
+          filename="${mesh_dir}/waist_Link.STL" />
       </geometry>
       <material
@@ -79,5 +86,5 @@
       <geometry>
         <mesh
-          filename="package://robotic_arm/meshes/waist_Link.STL" />
+          filename="${mesh_dir}/waist_Link.STL" />
       </geometry>
     </collision>
@@ -123,5 +130,5 @@
       <geometry>
         <mesh
-          filename="package://robotic_arm/meshes/arm_Link.STL" />
+          filename="${mesh_dir}/arm_Link.STL" />
       </geometry>
       <material
@@ -137,5 +144,5 @@
       <geometry>
         <mesh
-          filename="package://robotic_arm/meshes/arm_Link.STL" />
+          filename="${mesh_dir}/arm_Link.STL" />
       </geometry>
     </collision>
@@ -181,5 +188,5 @@
       <geometry>
         <mesh
-          filename="package://robotic_arm/meshes/end_Link.STL" />
+          filename="${mesh_dir}/end_Link.STL" />
       </geometry>
       <material
@@ -195,5 +202,5 @@
       <geometry>
         <mesh
-          filename="package://robotic_arm/meshes/end_Link.STL" />
+          filename="${mesh_dir}/end_Link.STL" />
       </geometry>
     </collision>
@@ -239,5 +246,5 @@
       <geometry>
         <mesh
-          filename="package://robotic_arm/meshes/support_Link.STL" />
+          filename="${mesh_dir}/support_Link.STL" />
       </geometry>
       <material
@@ -253,5 +260,5 @@
       <geometry>
         <mesh
-          filename="package://robotic_arm/meshes/support_Link.STL" />
+          filename="${mesh_dir}/support_Link.STL" />
       </geometry>
     </collision>
@@ -292,5 +299,5 @@
       <geometry>
         <mesh
-          filename="package://robotic_arm/meshes/cam_Link.STL" />
+          filename="${mesh_dir}/cam_Link.STL" />
       </geometry>
       <material
@@ -306,5 +313,5 @@
       <geometry>
         <mesh
-          filename="package://robotic_arm/meshes/cam_Link.STL" />
+          filename="${mesh_dir}/cam_Link.STL" />
       </geometry>
     </collision>
@@ -342,8 +349,10 @@
       <joint name="${joint}_joint">
         <hardwareInterface>position</hardwareInterface>
+        <hardwareInterface>velocity</hardwareInterface>
         <mechanicalReduction>1.0</mechanicalReduction>
       </joint>
       <actuator name="${joint}_motor">
         <hardwareInterface>position</hardwareInterface>
+        <hardwareInterface>velocity</hardwareInterface>
         <mechanicalReduction>1.0</mechanicalReduction>
       </actuator>
@@ -360,25 +369,52 @@
         <child link="cam_Link_optical"/>
     </joint>
+    <xacro:if value="${use_ignition}">
+      <gazebo reference="cam_Link">
+        <sensor name="camera_sensor" type="camera">
+          <camera>
+            <horizontal_fov>1.3962634</horizontal_fov>
+            <image>
+              <width>1280</width>
+              <height>1280</height>
+            </image>
+            <clip>
+              <near>0.1</near>
+              <far>100</far>
+            </clip>
+          </camera>
+          <plugin name="ignition::ros_camera_system" filename="libignition_ros_camera_system.so">
+            <ros>
+              <namespace>/</namespace>
+              <remapping>image_raw:=/camera/image_raw</remapping>
+            </ros>
+            <camera_name>cam</camera_name>
+            <frame_name>cam_link_optical</frame_name>
+          </plugin>
+        </sensor>
+      </gazebo>
+    </xacro:if>
+    <xacro:unless value="${use_ignition}">
     <gazebo reference="cam_Link">
-        <material>Gazebo/Red</material>
-        <sensor name="camera_sensor" type="camera">
-            <pose>0 0 0 0 0 0</pose>
-            <visualize>true</visualize>
-            <update_rate>10.0</update_rate>
-            <camera name="cam">
-              <horizontal_fov>1.3962634</horizontal_fov>
-              <image>
-                <width>1280</width>
-                <height>1280</height>
-                <format>R8G8B8</format>
-              </image>
-            </camera>
-            <plugin name="camera_controller" filename="libgazebo_ros_camera.so">
-                <frame_name>cam_link_optical</frame_name>
-                <image_width>1280</image_width>
-                <image_height>1280</image_height>
-                <update_rate>10.0</update_rate>
-            </plugin>
-        </sensor>
+      <material>Gazebo/Red</material>
+      <sensor name="camera_sensor" type="camera">
+        <pose>0 0 0 0 0 0</pose>
+        <visualize>true</visualize>
+        <update_rate>10.0</update_rate>
+        <camera name="cam">
+          <horizontal_fov>1.3962634</horizontal_fov>
+          <image>
+            <width>1280</width>
+            <height>1280</height>
+            <format>R8G8B8</format>
+          </image>
+        </camera>
+        <plugin name="camera_controller" filename="libgazebo_ros_camera.so">
+          <frame_name>cam_link_optical</frame_name>
+          <image_width>1280</image_width>
+          <image_height>1280</image_height>
+          <update_rate>10.0</update_rate>
+        </plugin>
+      </sensor>
     </gazebo>
+  </xacro:unless>
 </robot>

File: robotic_arm/urdf/Robot_Arm_control.xacro (robot description, xacro)
@@ -2,8 +2,14 @@
 <robot name="robotic_arm" xmlns:xacro="http://www.ros.org/wiki/xacro">
     <ros2_control name="RobotSystem" type="system">
-        <hardware>
-            <!-- By default, set up controllers for simulation. This won't work on real hardware -->
-            <plugin>gazebo_ros2_control/GazeboSystem</plugin>
-        </hardware>
+        <xacro:if value="${use_ignition}">
+            <hardware>
+                <plugin>ign_ros2_control/IgnitionSystem</plugin>
+            </hardware>
+        </xacro:if>
+        <xacro:unless value="${use_ignition}">
+            <hardware>
+                <plugin>gazebo_ros2_control/GazeboSystem</plugin>
+            </hardware>
+        </xacro:unless>
         <joint name="base_waist_joint">
             <command_interface name="position">
@@ -11,4 +17,6 @@
                 <param name="max">3.142/2</param>
             </command_interface>
+            <command_interface name="velocity"/>
+            <state_interface name="velocity"/>
             <state_interface name="position"/>
         </joint>
@@ -18,4 +26,6 @@
                 <param name="max">3.142/2</param>
             </command_interface>
+            <command_interface name="velocity"/>
+            <state_interface name="velocity"/>
             <state_interface name="position"/>
         </joint>
@@ -25,4 +35,6 @@
                 <param name="max">3.142/2</param>
             </command_interface>
+            <command_interface name="velocity"/>
+            <state_interface name="velocity"/>
             <state_interface name="position"/>
         </joint>

File: robotic_arm/urdf/Robot_Arm_gazebo.xacro (robot description, xacro)
@@ -1,10 +1,19 @@
 <?xml version="1.0" encoding="utf-8"?>
 <robot name="robotic_arm" xmlns:xacro="http:///www.ros.org/wiki/xacro">
-  <gazebo>
-    <plugin name="gazebo_ros2_control" filename="libgazebo_ros2_control.so">
-      <robot_param>robot_description</robot_param>
-      <robot_param_node>robot_state_publisher</robot_param_node>
-      <parameters>$(find moveit_robotic_arm)/config/ros2_controllers.yaml</parameters>
-    </plugin>
-  </gazebo>
+  <xacro:if value="${use_ignition}">
+    <plugin name="ign_ros2_control::IgnitionROS2ControlPlugin" filename="ign_ros2_control-system">
+        <robot_param>robot_description</robot_param>
+        <robot_param_node>robot_state_publisher</robot_param_node>
+        <parameters>$(find moveit_robotic_arm)/config/ros2_controllers.yaml</parameters>
+      </plugin>
+  </xacro:if>
+  <xacro:unless value="${use_ignition}">
+    <gazebo>
+      <plugin name="gazebo_ros2_control" filename="libgazebo_ros2_control.so">
+        <robot_param>robot_description</robot_param>
+        <robot_param_node>robot_state_publisher</robot_param_node>
+        <parameters>$(find moveit_robotic_arm)/config/ros2_controllers.yaml</parameters>
+      </plugin>
+    </gazebo>
+  </xacro:unless>
 </robot>

Commit message: error fix

File: robotic_arm/urdf/Robot_Arm.xacro (robot description, xacro)
@@ -2,6 +2,6 @@
 <robot name="robotic_arm" xmlns:xacro="http:///www.ros.org/wiki/xacro">
   <xacro:property name="use_ignition" default="false"/>
-  <xacro:include filename="$(find robotic_arm)/urdf/Robot_Arm_control.xacro"/>
-  <xacro:include filename="$(find robotic_arm)/urdf/Robot_Arm_gazebo.xacro"/>
+  <xacro:include filename="$(find robotic_arm)/urdf/Robot_Arm_control.xacro" />
+  <xacro:include filename="$(find robotic_arm)/urdf/Robot_Arm_gazebo.xacro" />
   <xacro:if value="${use_ignition}">
     <xacro:property name="mesh_dir" value="/home/khaled/ros2_ws/src/robotic_arm/meshes"/>
@@ -369,51 +369,26 @@
         <child link="cam_Link_optical"/>
     </joint>
-    <xacro:if value="${use_ignition}">
-      <gazebo reference="cam_Link">
+  <xacro:unless value="${use_ignition}">
+    <gazebo reference="cam_Link">
+        <material>Gazebo/Red</material>
         <sensor name="camera_sensor" type="camera">
-          <camera>
-            <horizontal_fov>1.3962634</horizontal_fov>
-            <image>
-              <width>1280</width>
-              <height>1280</height>
-            </image>
-            <clip>
-              <near>0.1</near>
-              <far>100</far>
-            </clip>
-          </camera>
-          <plugin name="ignition::ros_camera_system" filename="libignition_ros_camera_system.so">
-            <ros>
-              <namespace>/</namespace>
-              <remapping>image_raw:=/camera/image_raw</remapping>
-            </ros>
-            <camera_name>cam</camera_name>
-            <frame_name>cam_link_optical</frame_name>
-          </plugin>
+            <pose>0 0 0 0 0 0</pose>
+            <visualize>true</visualize>
+            <update_rate>10.0</update_rate>
+            <camera name="cam">
+              <horizontal_fov>1.3962634</horizontal_fov>
+              <image>
+                <width>1280</width>
+                <height>1280</height>
+                <format>R8G8B8</format>
+              </image>
+            </camera>
+            <plugin name="camera_controller" filename="libgazebo_ros_camera.so">
+                <frame_name>cam_link_optical</frame_name>
+                <image_width>1280</image_width>
+                <image_height>1280</image_height>
+                <update_rate>10.0</update_rate>
+            </plugin>
         </sensor>
-      </gazebo>
-    </xacro:if>
-    <xacro:unless value="${use_ignition}">
-    <gazebo reference="cam_Link">
-      <material>Gazebo/Red</material>
-      <sensor name="camera_sensor" type="camera">
-        <pose>0 0 0 0 0 0</pose>
-        <visualize>true</visualize>
-        <update_rate>10.0</update_rate>
-        <camera name="cam">
-          <horizontal_fov>1.3962634</horizontal_fov>
-          <image>
-            <width>1280</width>
-            <height>1280</height>
-            <format>R8G8B8</format>
-          </image>
-        </camera>
-        <plugin name="camera_controller" filename="libgazebo_ros_camera.so">
-          <frame_name>cam_link_optical</frame_name>
-          <image_width>1280</image_width>
-          <image_height>1280</image_height>
-          <update_rate>10.0</update_rate>
-        </plugin>
-      </sensor>
     </gazebo>
   </xacro:unless>

File: robotic_arm/urdf/Robot_Arm_control.xacro (robot description, xacro)
@@ -18,6 +18,6 @@
             </command_interface>
             <command_interface name="velocity"/>
+            <state_interface name="position"/>
             <state_interface name="velocity"/>
-            <state_interface name="position"/>
         </joint>
         <joint name="waist_arm_joint">

File: robotic_arm/urdf/Robot_Arm_gazebo.xacro (robot description, xacro)
@@ -2,9 +2,11 @@
 <robot name="robotic_arm" xmlns:xacro="http:///www.ros.org/wiki/xacro">
   <xacro:if value="${use_ignition}">
-    <plugin name="ign_ros2_control::IgnitionROS2ControlPlugin" filename="ign_ros2_control-system">
+    <gazebo>
+      <plugin name="ign_ros2_control::IgnitionROS2ControlPlugin" filename="ign_ros2_control-system">
         <robot_param>robot_description</robot_param>
         <robot_param_node>robot_state_publisher</robot_param_node>
         <parameters>$(find moveit_robotic_arm)/config/ros2_controllers.yaml</parameters>
       </plugin>
+    </gazebo>
   </xacro:if>
   <xacro:unless value="${use_ignition}">
